File: _autosave-main.kicad_sch (KiCad schematic)
At the start: 0 parts

Commit message: my first push
Other:
- title: Design project -> (none)
Changed lines of the file:
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@@
 	(paper "A4")
 	(title_block
-		(title "Design project")
 		(date "2025-03-23")
 		(rev "v0")
@@
 		(comment 4 "Phila Haanyama, Hannah Owen")
 	)
-	(sheet_instances
-		(path "/"
-			(page "1")
-		)
-	)
-	(embedded_fonts no)
 )
