File: EEE3088F Design project.kicad_sch (KiCad schematic)
At the start: 2 parts, among them J1 Conn_02x16_Odd_Even, J4 Conn_01x02

Commit message: Removed old backups and updated KiCad files
Parts:
- added C27: 10uF, Capacitor_SMD:C_0805_2012Metric_Pad1.18x1.45mm_HandSolder, symbol Device:C_Small
- added C28, C32, C40, C41, C42, C46, C48, C50, C51: 100uF, Capacitor_SMD:C_1206_3216Metric_Pad1.33x1.80mm_HandSolder, symbol Device:C_Small
- added C34: 0.1uF, Capacitor_SMD:C_0402_1005Metric_Pad0.74x0.62mm_HandSolder, symbol Device:C_Small
- added C43: 47nF, Capacitor_SMD:C_0603_1608Metric_Pad1.08x0.95mm_HandSolder, symbol Device:C_Small
- added C44: 1nF, Capacitor_SMD:C_0603_1608Metric_Pad1.08x0.95mm_HandSolder, symbol Device:C_Small
- added C45, C47, C49: 22uF, Capacitor_SMD:C_0805_2012Metric_Pad1.18x1.45mm_HandSolder, symbol Device:C_Small
- added D3: D_Schottky, Diode_SMD:D_SOD-123, symbol Device:D_Schottky
- added L3: 22uH, Inductor_SMD:L_0603_1608Metric_Pad1.05x0.95mm_HandSolder, symbol Device:L_Small
- added L6: 1.2uH, Inductor_SMD:L_0805_2012Metric_Pad1.05x1.20mm_HandSolder, symbol Device:L_Small
- added Q3: NMOS, Package_TO_SOT_SMD:SOT-23, symbol Simulation_SPICE:NMOS
- added R21: 5.1k, Resistor_SMD:R_0805_2012Metric_Pad1.20x1.40mm_HandSolder, symbol Device:R_Small_US
- added R27: 390, Resistor_SMD:R_0603_1608Metric_Pad0.98x0.95mm_HandSolder, symbol Device:R_Small_US
- added R28: 1k, Resistor_SMD:R_0603_1608Metric_Pad0.98x0.95mm_HandSolder, symbol Device:R_Small_US
- added R29: 10k, Resistor_SMD:R_0805_2012Metric_Pad1.20x1.40mm_HandSolder, symbol Device:R_Small_US
- added R30: 2.7k, Resistor_SMD:R_0805_2012Metric_Pad1.20x1.40mm_HandSolder, symbol Device:R_Small_US
- added R31: 220K, Resistor_SMD:R_0603_1608Metric_Pad0.98x0.95mm_HandSolder, symbol Device:R_Small_US
- added R32: 33K, Resistor_SMD:R_0603_1608Metric_Pad0.98x0.95mm_HandSolder, symbol Device:R_Small_US
- added R33: 100K, Resistor_SMD:R_0402_1005Metric_Pad0.72x0.64mm_HandSolder, symbol Device:R_Small_US
- added R34: 68K, Resistor_SMD:R_0603_1608Metric_Pad0.98x0.95mm_HandSolder, symbol Device:R_Small_US
- added R35: 150K, Resistor_SMD:R_0805_2012Metric_Pad1.20x1.40mm_HandSolder, symbol Device:R_Small_US
- added R36: 47K, Resistor_SMD:R_0805_2012Metric_Pad1.20x1.40mm_HandSolder, symbol Device:R_Small_US
- added SW2: SW_SPDT, SWITCH:Untitled, symbol Switch:SW_SPDT
- added TP20, TP30, TP31, TP32, TP33, TP44: TestPoint, TestPoint:TestPoint_Pad_1.0x1.0mm, symbol Connector:TestPoint
- added U10: TPS61088RHLR, TPS61088RHLR:TPS61088RHLR, symbol TPS61088RHLR:TPS61088RHLR
- added U13, U14: RT9742CGJ5, Package_TO_SOT_SMD:TSOT-23-5, symbol HIGH SIDE SWITCH:RT9742CGJ5
- added U6: XL1509-3.3, Package_SO:SOIC-8_3.9x4.9mm_P1.27mm, symbol Regulator_Switching:XL1509-3.3
Connections:
- net 3V3_Out: now also C46.1, C48.1, C50.1, C51.1, L3.2, TP33.1, U6.3 (FB)
- net 5V_Out: now also C28.1, C32.1, C40.1, C41.1, C42.1, C45.2, C47.2, C49.2, R35.2, TP31.1, TP32.1, U10.15 (VOUT_14), U13.5 (VIN), U14.5 (VIN), U6.1 (VIN)
- net CTRL_EXT_LOAD1: now also U13.4 (EN)
- net CTRL_EXT_LOAD2: now also U14.4 (EN)
- net EXT_LOAD1_OUT: now also U13.1 (VOUT)
- net EXT_LOAD2_OUT: now also U14.1 (VOUT)
- net FAST_CHARGE_CTRL: now also R28.2
- net GND: now also C27.2, C28.2, C32.2, C40.2, C41.2, C42.2, C43.2, C44.2, C45.1, C46.2, C47.1, C48.2, C49.1, C50.2, C51.2, D3.2 (A), Q3.3 (S), R27.2, R29.2, R33.1, R36.1, TP20.1, U10.1 (VCC), U10.20 (AGND), U10.21 (PGND), U13.2 (GND), U14.2 (GND), U6.4 (~{EN}), U6.5 (GND), U6.6 (GND), U6.7 (GND), U6.8 (GND)
- new net: R33.2, U10.19 (ILIM)
- new net: C43.1, U10.10 (SS)
- new net: R34.2, U10.18 (COMP)
- new net: R32.2, U10.3 (FSW)
- new net: C34.1, L6.2, R31.1, U10.5 (SW_4)
- new net: C34.2, U10.8 (BOOT)
- new net: C44.1, R34.1
- new net: R21.2, R27.1
- new net: Q3.2 (G), R28.1, R29.1
- new net: R31.2, R32.1
- new net: Q3.1 (D), R30.2
- new net: D3.1 (K), L3.1, U6.2 (OUT)
- new net FB: R35.1, R36.2, TP44.1, U10.17 (FB)
- new net VCC: SW2.2 (B)
- new net Vprog: R21.1, R30.1
- new net Vswitch: C27.1, L6.1, SW2.1 (A), TP30.1, U10.2 (EN), U10.9 (VIN)
Other:
- sheet 3V3 5V output renamed 3V3 and 5V output
- sheet battery renamed Battery
- sheet external load switch renamed External load switching system
- note added: "3V3 AND 5V OUTPUT SCHEMATIC"
- note added: "3V3 BUCK CONVERTER SCHEMATIC"
- note added: "5V BOOST CONVERTER SCHEMATIC"
- note added: "Connected to IN- of INA219"
- note added: "Connected to PROG pin of battery charger"
- note added: "Connected to pin13 of connector. Determines HIGH or LOW current mode"
- note added: "DUAL-MODE BATTERY CHARGER SCHEMATIC"
- note added: "EN connected to pin25. Switches ON/OFF the external load connection"
- note added: "EN connected to pin7. Switches ON/OFF the external load connection"
- note added: "EXTERNAL LOAD SWITCHING 1"
- note added: "EXTERNAL LOAD SWITCHING 2"
- note added: "EXTERNAL LOAD SWITCHING SCHEMATIC"
- note added: "FB connected to voltage divider R25 and R26"
- note added: "FLG intentionally left unconnected"
- note added: "MODE, SW_5, SW_6, SW_7, VOUT_15, VOUT_16, NC_11 and NC_12 are intentionally left unconnected"
- note added: "ON/OFF SWITCH SCHEMATIC"
- note added: "OUT connected to pin18 of connector. Ideal output voltage is 3V3"
- note added: "Pin1 Connected to VIN and EN on the 5V boost converter"
- note added: "Pin3 intentionally left unconnected"
- note added: "R14 and R15 determine value of current when pin13 of connector is LOW switching OFF NMOS"
- note added: "R18 reduces current entering NMOS"
- note added: "R19 is a pull down resistor"
- note added: "R20 and R22 connected to FSW determine switching frequency"
- note added: "R24 connected to ILIM determines peak current value"
- note added: "R25 and R26 determine value of output voltage"
- note added: "The parallel combination of R14 and R15 with R16 determines value of current when pin13 of connector is HIGH switching ON NMOS"
- note added: "VIN and EN connected to pin1 of switch"
- note added: "VIN connected to pin20 of connector."
- note added: "VOUT connected to pin11 of connector"
- note added: "VOUT connected to pin21 of connector"
- note added: "VOUT_14 connected to pin20 of connector. Ideal output voltage is 5V"
- note added: "Vin connected to pin20 of connector"
- note added: "Voltage divider output connected to FB"
- title: Design project -> MICRO-MOUSE POWER SUBSYSTEM
- moved on the sheet: J1, J4

Commit message: added comments
Parts:
- added C10: 2.2μ, Capacitor_SMD:C_1210_3225Metric_Pad1.33x2.70mm_HandSolder, symbol CL31B225KBHNNNE[1]:CL31B225KBHNNNE
- added C11, C8: 10μ, Capacitor_SMD:C_0805_2012Metric_Pad1.18x1.45mm_HandSolder, symbol CL21A106KAYNNNE[1]:CL21A106KAYNNNE
- added C52, C53, C54, C55, C56, C57, C58, C59: 100uF, Capacitor_SMD:C_1206_3216Metric_Pad1.33x1.80mm_HandSolder, symbol Device:C_Small
- added C60: 100n, Capacitor_SMD:C_0402_1005Metric_Pad0.74x0.62mm_HandSolder, symbol CL05B104KO5NNNC[1]:CL05B104KO5NNNC
- added C61, C9: 10n, Capacitor_SMD:C_0603_1608Metric_Pad1.08x0.95mm_HandSolder, symbol 0603B103K500NT[1]:0603B103K500NT
- added C62: 2.2μ, Capacitor_SMD:C_1206_3216Metric_Pad1.33x1.80mm_HandSolder, symbol CL31B225KBHNNNE[1]:CL31B225KBHNNNE
- added D4: D_Schottky, Diode_SMD:D_SOD-123, symbol Device:D_Schottky
- added J5: HUSB237, Package_DFN_QFN:DFN-6-1EP_2x2mm_P0.65mm_EP1x1.6mm, symbol 54-00285[1]:54-00285
- added J6: 54-00285, Connector_USB:USB_C_Receptacle_HRO_TYPE-C-31-M-17, symbol 54-00285[1]:54-00285
- added L4: 22uH, Inductor_SMD:L_0603_1608Metric_Pad1.05x0.95mm_HandSolder, symbol Device:L_Small
- added R37, R38, R43, R46: 10k, Resistor_SMD:R_1206_3216Metric_Pad1.30x1.75mm_HandSolder, symbol 1206W4F1002T5E[1]:1206W4F1002T5E
- added R39: 0.05, Resistor_SMD:R_1206_3216Metric_Pad1.30x1.75mm_HandSolder, symbol RL1206FR-070R05L[1]:RL1206FR-070R05L
- added R40: 75k, Resistor_SMD:R_1206_3216Metric_Pad1.30x1.75mm_HandSolder, symbol 1206W4F1002T5E[1]:1206W4F1002T5E
- added R41, R42: 0.4, Resistor_SMD:R_1206_3216Metric_Pad1.30x1.75mm_HandSolder, symbol 1206W4F400LT5E[1]:1206W4F400LT5E
- added R44: 1, Resistor_SMD:R_1206_3216Metric_Pad1.30x1.75mm_HandSolder, symbol 1206W4F100KT5E[1]:1206W4F100KT5E
- added R45: 1, Resistor_SMD:R_1206_3216Metric_Pad1.30x1.75mm_HandSolder, symbol 1206W4F400LT5E[1]:1206W4F400LT5E
- added TP45, TP46, TP47, TP48, TP49, TP50, TP51, TP52, TP53, TP54, TP55, TP56, TP57, TP58, TP59, TP60, TP61, TP62, TP63, TP64, TP65, TP66, TP67, TP68, TP69, TP70, TP71, TP72, TP73, TP74: TestPoint, TestPoint:TestPoint_Pad_1.0x1.0mm, symbol Connector:TestPoint
- added U15: XL1509-5.0, Package_SO:SOIC-8_3.9x4.9mm_P1.27mm, symbol Regulator_Switching:XL1509-5.0
- added U16, U18: INA219AIDR, Package_SO:SOIC-8_3.9x4.9mm_P1.27mm, symbol INA219AIDR[1]:INA219AIDR
- added U17: auxilliary motors, Package_SO:HTSSOP-16-1EP_4.4x5mm_P0.65mm_EP3.4x5mm_Mask2.46x2.31mm, symbol DRV8833PWPR[1]:DRV8833PWPR
- added U3: Primary motors, Package_SO:HTSSOP-16-1EP_4.4x5mm_P0.65mm_EP3.4x5mm_Mask2.46x2.31mm, symbol DRV8833PWPR[1]:DRV8833PWPR
Connections:
- net 3V3_Out: now also C60.2, TP70.1, U16.1 (A1), U17.1 (NSLEEP), U3.1 (NSLEEP)
- net 5V_Out: now also C11.1, C61.2, C8.1, C9.2, TP45.1, TP54.1, U17.12 (VM), U3.12 (VM)
- net Battery: now also R39.1, TP69.1, U16.8 (VIN+)
- net GND: now also C10.2, C11.2, C52.2, C53.2, C54.2, C55.2, C56.2, C57.2, C58.2, C59.2, C62.2, C8.2, D4.2 (A), J5.7 (GND), J6.A12 (GND_A), J6.B12 (GND_B), J6.S1 (EH), R40.1, R41.2, R42.2, R44.2, R45.2, U15.4 (~{EN}), U15.5 (GND), U15.6 (GND), U15.7 (GND), U15.8 (GND), U16.2 (A0), U16.6 (GND), U17.13 (GND), U3.13 (GND)
- net HV: now also C52.1, C53.1, C54.1, C55.1, C56.1, J5.2 (VBUS), J6.A9 (VBUS_A), J6.B9 (VBUS_B), TP74.1, U15.1 (VIN)
- net I2C1_SCL: now also R37.1
- net I2C1_SDA: now also R38.1
- net MOTOR1_A_OUT: now also TP53.1, U3.2 (AOUT1)
- net MOTOR1_B_OUT: now also TP52.1, U3.4 (AOUT2)
- net MOTOR1_CTRL1: now also TP48.1, U3.16 (AIN1)
- net MOTOR1_CTRL2: now also TP46.1, U3.15 (AIN2)
- net MOTOR2_A_OUT: now also TP67.1, U3.7 (BOUT1)
- net MOTOR2_B_OUT: now also TP51.1, U3.5 (BOUT2)
- net MOTOR2_CTRL1: now also TP49.1, U3.9 (BIN1)
- net MOTOR2_CTRL2: now also TP47.1, U3.10 (BIN2)
- net MOTOR3_A_OUT: now also TP60.1, U17.2 (AOUT1)
- net MOTOR3_B_OUT: now also TP63.1, U17.4 (AOUT2)
- net MOTOR3_CTRL1: now also TP55.1, U17.16 (AIN1)
- net MOTOR3_CTRL2: now also TP57.1, U17.15 (AIN2)
- net MOTOR4_A_OUT: now also TP62.1, U17.7 (BOUT1)
- net MOTOR4_B_OUT: now also TP61.1, U17.5 (BOUT2)
- net MOTOR4_CTRL1: now also TP56.1, U17.9 (BIN1)
- net MOTOR4_CTRL2: now also TP58.1, U17.10 (BIN2)
- net VCC: now also R39.2, U16.7 (VIN-)
- new net: C57.1, C58.1, C59.1, L4.2, TP73.1
- new net: D4.1 (K), L4.1, U15.2 (OUT)
- new net: J6.A5 (CC1), R43.2
- new net: J6.B5 (CC2), R46.2
- new net: C60.1, TP72.1, U16.5 (VS)
- new net: R38.2, TP71.1, U16.3 (SDA)
- new net: C62.1, U17.14 (VINT)
- new net: R45.1, U3.6 (BISEN)
- new net: TP59.1, U17.8 (~{NFAULT})
- new net: C61.1, U17.11 (VCP)
- new net: R44.1, U3.3 (AISEN)
- new net: C10.1, U3.14 (VINT)
- new net: R42.1, U17.6 (BISEN)
- new net: J5.3 (VSET), R40.2, TP64.1
- new net: R41.1, U17.3 (AISEN)
- new net: TP50.1, U3.8 (~{NFAULT})
- new net: C9.1, U3.11 (VCP)
- new net: R37.2, TP68.1, U16.4 (SCL)
- new net CC1: J5.1 (CC1), R43.1, TP65.1
- new net CC2: J5.6 (CC2), R46.1, TP66.1
Other:
- note added: "6 pin USB-C connector"
- note added: "9 V input from USB"
- note added: "A0 and A1 can't both be connected to GND so A1 is tied to logic high"
- note added: "AIN pins controls input of 1 motor and BIN pins control input of other motor"
- note added: "AOUT controls output to 1 motor and BOUT controls output to other motor"
- note added: "Capacitors added for stability parallel configuration in order to get a total capacitance of 500 uF"
- note added: "Charging battery with 9 V"
- note added: "Data of readings from INA219 sent to motherboard"
- note added: "INA219 Connection"
- note added: "INA219 connected to battery so it can take voltage readings"
- note added: "Motor Connections"
- note added: "Motors powered by 5 V power rail"
- note added: "NSleep connected to 3V3 so that IC stays enabled during operation"
- note added: "Powered by 3V3 output from 2x16 connecotr"
- note added: "Resistor to set the output to 9 V"
- note added: "Resistors to set output current to motors"
- note added: "Spare INA219"
- note added: "Test points to measure voltage at the inputs and outputs"
- note added: "To test that 4.2 V is going to the battery"
- note added: "USB-C Connector"
- note added: "USB-C Power delivery IC"
- note added: "VBus pins tied together so USB orientation doesn't matter"
- note added: "connected to HV pin of the 2x16 connector"
- note added: "enable pin driven low to turn on device"
- note added: "logic low when faulty"
- note added: "regulated output"
- note added: "shunt resistor used to measure current coming from battery"
- note added: "test points to measure if 3V3 out is powering INA219 correctly"
- moved on the sheet: C27, C28, C32, C34, C40, C41, C42, C43, C44, C45, C46, C47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
